File: RegMouthJarPCBA/RegMouthJarPCBA.sch (KiCad schematic (older format))
At the start: 8 parts, among them CON1 BARREL_JACK, J1 4P4C, J2 4P4C, K1 CONN_3, P2 CONN_4, P3 CONN_4

Commit message: adding temperature test point
Parts:
- added P101: CONN_2, symbol CONN_2
Other:
- note added: "Pinout:\n1: V+\n2: V-"
- note added: "Temperature test point"
Changed lines of the file:
@@
 	3400 2800 3400 2550
 Connection ~ 3300 2800
+$Comp
+L CONN_2 P101
+U 1 1 539131C2
+P 8800 2450
+F 0 "P101" V 8750 2450 40  0000 C CNN
+F 1 "CONN_2" V 8850 2450 40  0000 C CNN
+F 2 "" H 8800 2450 60  0000 C CNN
+F 3 "" H 8800 2450 60  0000 C CNN
+	1    8800 2450
+	0    -1   -1   0
+$EndComp
+Text Notes 8400 2100 0    60   ~ 0
+Temperature test point
+Text Notes 9050 2300 0    40   ~ 0
+Pinout:\n1: V+\n2: V-
 $EndSCHEMATC

Commit message: tweaking board layout.
Parts:
- renumbered K1 to P1, P101 to P4
Connections:
- wire segments 29 -> 31
Changed lines of the file:
@@
 Text Notes 7150 1650 0    40   ~ 0
 Pinout:\n1: My RX, Your TX\n2: GND\n3: GND\n4: My TX, Your RX
-$Comp
-L GND #PWR02
-U 1 1 5391240D
-P 6700 2550
-F 0 "#PWR02" H 6700 2550 30  0001 C CNN
-F 1 "GND" H 6700 2480 30  0001 C CNN
-F 2 "" H 6700 2550 60  0000 C CNN
-F 3 "" H 6700 2550 60  0000 C CNN
-	1    6700 2550
-	1    0    0    -1
-$EndComp
-$Comp
-L GND #PWR03
-U 1 1 5391241C
-P 6850 2550
-F 0 "#PWR03" H 6850 2550 30  0001 C CNN
-F 1 "GND" H 6850 2480 30  0001 C CNN
-F 2 "" H 6850 2550 60  0000 C CNN
-F 3 "" H 6850 2550 60  0000 C CNN
-	1    6850 2550
-	1    0    0    -1
-$EndComp
-$Comp
-L GND #PWR04
-U 1 1 5391242B
-P 7450 2550
-F 0 "#PWR04" H 7450 2550 30  0001 C CNN
-F 1 "GND" H 7450 2480 30  0001 C CNN
-F 2 "" H 7450 2550 60  0000 C CNN
-F 3 "" H 7450 2550 60  0000 C CNN
-	1    7450 2550
-	1    0    0    -1
-$EndComp
-$Comp
-L GND #PWR05
-U 1 1 5391243A
-P 7550 2550
-F 0 "#PWR05" H 7550 2550 30  0001 C CNN
-F 1 "GND" H 7550 2480 30  0001 C CNN
-F 2 "" H 7550 2550 60  0000 C CNN
-F 3 "" H 7550 2550 60  0000 C CNN
-	1    7550 2550
-	1    0    0    -1
-$EndComp
-Wire Wire Line
-	7450 2450 7450 2550
-Wire Wire Line
-	7550 2450 7550 2550
-Wire Wire Line
-	6700 2450 6700 2550
-Wire Wire Line
-	6850 2450 6850 2550
-Wire Wire Line
-	6600 2450 6600 2700
-Wire Wire Line
-	6600 2700 7350 2700
-Wire Wire Line
-	7350 2700 7350 2450
-Wire Wire Line
-	6950 2450 6950 2800
-Wire Wire Line
-	6950 2800 7650 2800
-Wire Wire Line
-	7650 2800 7650 2450
 Text Notes 3200 1800 0    40   ~ 0
 Pinout:\n1: V+\n2: AGND\n3: PWRGND
 $Comp
-L CONN_3 K1
+L CONN_3 P1
 U 1 1 539126EB
 P 3300 2200
-F 0 "K1" V 3250 2200 50  0000 C CNN
+F 0 "P1" V 3250 2200 50  0000 C CNN
 F 1 "CONN_3" V 3350 2200 40  0000 C CNN
 F 2 "" H 3300 2200 60  0000 C CNN
@@
 Connection ~ 3300 2800
 $Comp
-L CONN_2 P101
+L CONN_2 P4
 U 1 1 539131C2
 P 8800 2450
-F 0 "P101" V 8750 2450 40  0000 C CNN
+F 0 "P4" V 8750 2450 40  0000 C CNN
 F 1 "CONN_2" V 8850 2450 40  0000 C CNN
 F 2 "" H 8800 2450 60  0000 C CNN
@@
 Text Notes 9050 2300 0    40   ~ 0
 Pinout:\n1: V+\n2: V-
+Wire Wire Line
+	6600 2450 6600 2550
+Wire Wire Line
+	6600 2550 7350 2550
+Wire Wire Line
+	7350 2550 7350 2450
+Wire Wire Line
+	6700 2450 6700 2650
+Wire Wire Line
+	6700 2650 7450 2650
+Wire Wire Line
+	7450 2650 7450 2450
+Wire Wire Line
+	6850 2450 6850 2750
+Wire Wire Line
+	6850 2750 7550 2750
+Wire Wire Line
+	7550 2750 7550 2450
+Wire Wire Line
+	6950 2450 6950 2850
+Wire Wire Line
+	6950 2850 7650 2850
+Wire Wire Line
+	7650 2850 7650 2450
 $EndSCHEMATC
