File: RegMouthJarPCBA/RegMouthJarPCBA.kicad_pcb (KiCad board)
At the start: 2 copper layers, 68.1 x 68.1 mm, 10 parts, among them CON1 BARREL_JACK, J1 4P4C, J2 4P4C, P1 CONN_3, P2 CONN_4, P3 CONN_4, P4 CONN_2

Commit message: bulk update.  starting tweaks for v2.
Parts:
- P2, P3: moved to B.Cu
Other:
- board text added: "(v2)"
- board text added: "9V to 24V DC"
- board text added: "Force+"
- board text added: "Force-"
- board text added: "GND"
- board text added: "RX (Your TX)"
- board text added: "Sense+"
- board text added: "Sense-"
- board text added: "TX (Your RX)"
- board text removed: "(v1)"
Changed lines of the file:
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@@
     (area 185.42 133.985 256.540001 205.105001)
     (thickness 1.6)
-    (drawings 17)
+    (drawings 26)
     (tracks 35)
     (zones 0)
@@
     (mod_text_size 1 1)
     (mod_text_width 0.15)
-    (pad_size 1.5 1.5)
-    (pad_drill 0.6)
+    (pad_size 3.2 3.2)
+    (pad_drill 3.2)
     (pad_to_mask_clearance 0)
     (aux_axis_origin 185.42 133.985)
@@
     (add_net N-000009)
   )
-  (module PIN_ARRAY_4x1 (layer F.Cu)
+  (module PIN_ARRAY_4x1 (layer B.Cu)
     (at 220.98 195.199)
     (descr "Double rangee de contacts 2 x 5 pins")
     (tags CONN)
-    (fp_text reference P3 (at 6.35 -0.254) (layer F.SilkS)
-      (effects (font (size 1.016 1.016) (thickness 0.2032)))
-    )
-    (fp_text value CONN_4 (at 0 2.54) (layer F.SilkS) hide
-      (effects (font (size 1.016 1.016) (thickness 0.2032)))
-    )
-    (fp_line (start 5.08 1.27) (end -5.08 1.27) (layer F.SilkS) (width 0.254))
-    (fp_line (start 5.08 -1.27) (end -5.08 -1.27) (layer F.SilkS) (width 0.254))
-    (fp_line (start -5.08 -1.27) (end -5.08 1.27) (layer F.SilkS) (width 0.254))
-    (fp_line (start 5.08 1.27) (end 5.08 -1.27) (layer F.SilkS) (width 0.254))
+    (fp_text reference P3 (at 6.35 0.254) (layer B.SilkS)
+      (effects (font (size 0.762 0.762) (thickness 0.1524)) (justify mirror))
+    )
+    (fp_text value CONN_4 (at 0 -2.54) (layer B.SilkS) hide
+      (effects (font (size 1.016 1.016) (thickness 0.2032)) (justify mirror))
+    )
+    (fp_line (start 5.08 -1.27) (end -5.08 -1.27) (layer B.SilkS) (width 0.254))
+    (fp_line (start 5.08 1.27) (end -5.08 1.27) (layer B.SilkS) (width 0.254))
+    (fp_line (start -5.08 1.27) (end -5.08 -1.27) (layer B.SilkS) (width 0.254))
+    (fp_line (start 5.08 -1.27) (end 5.08 1.27) (layer B.SilkS) (width 0.254))
     (pad 1 thru_hole rect (at -3.81 0) (size 1.524 1.524) (drill 1.016)
-      (layers *.Cu *.Mask F.SilkS)
+      (layers *.Cu *.Mask B.SilkS)
       (net 8 N-000007)
     )
     (pad 2 thru_hole circle (at -1.27 0) (size 1.524 1.524) (drill 1.016)
-      (layers *.Cu *.Mask F.SilkS)
+      (layers *.Cu *.Mask B.SilkS)
       (net 9 N-000008)
     )
     (pad 3 thru_hole circle (at 1.27 0) (size 1.524 1.524) (drill 1.016)
-      (layers *.Cu *.Mask F.SilkS)
+      (layers *.Cu *.Mask B.SilkS)
       (net 10 N-000009)
     )
     (pad 4 thru_hole circle (at 3.81 0) (size 1.524 1.524) (drill 1.016)
-      (layers *.Cu *.Mask F.SilkS)
+      (layers *.Cu *.Mask B.SilkS)
       (net 3 N-0000010)
     )
@@
     )
   )
-  (module PIN_ARRAY_4x1 (layer F.Cu)
+  (module PIN_ARRAY_4x1 (layer B.Cu)
     (at 222.25 160.655)
     (descr "Double rangee de contacts 2 x 5 pins")
     (tags CONN)
-    (fp_text reference P2 (at 6.35 0) (layer F.SilkS)
-      (effects (font (size 1.016 1.016) (thickness 0.2032)))
-    )
-    (fp_text value CONN_4 (at 0 2.54) (layer F.SilkS) hide
-      (effects (font (size 1.016 1.016) (thickness 0.2032)))
-    )
-    (fp_line (start 5.08 1.27) (end -5.08 1.27) (layer F.SilkS) (width 0.254))
-    (fp_line (start 5.08 -1.27) (end -5.08 -1.27) (layer F.SilkS) (width 0.254))
-    (fp_line (start -5.08 -1.27) (end -5.08 1.27) (layer F.SilkS) (width 0.254))
-    (fp_line (start 5.08 1.27) (end 5.08 -1.27) (layer F.SilkS) (width 0.254))
+    (fp_text reference P2 (at 6.35 0) (layer B.SilkS)
+      (effects (font (size 0.762 0.762) (thickness 0.1524)) (justify mirror))
+    )
+    (fp_text value CONN_4 (at 0 -2.54) (layer B.SilkS) hide
+      (effects (font (size 1.016 1.016) (thickness 0.2032)) (justify mirror))
+    )
+    (fp_line (start 5.08 -1.27) (end -5.08 -1.27) (layer B.SilkS) (width 0.254))
+    (fp_line (start 5.08 1.27) (end -5.08 1.27) (layer B.SilkS) (width 0.254))
+    (fp_line (start -5.08 1.27) (end -5.08 -1.27) (layer B.SilkS) (width 0.254))
+    (fp_line (start 5.08 -1.27) (end 5.08 1.27) (layer B.SilkS) (width 0.254))
     (pad 1 thru_hole rect (at -3.81 0) (size 1.524 1.524) (drill 1.016)
-      (layers *.Cu *.Mask F.SilkS)
+      (layers *.Cu *.Mask B.SilkS)
       (net 4 N-0000012)
     )
     (pad 2 thru_hole circle (at -1.27 0) (size 1.524 1.524) (drill 1.016)
-      (layers *.Cu *.Mask F.SilkS)
+      (layers *.Cu *.Mask B.SilkS)
       (net 5 N-0000013)
     )
     (pad 3 thru_hole circle (at 1.27 0) (size 1.524 1.524) (drill 1.016)
-      (layers *.Cu *.Mask F.SilkS)
+      (layers *.Cu *.Mask B.SilkS)
       (net 6 N-0000014)
     )
     (pad 4 thru_hole circle (at 3.81 0) (size 1.524 1.524) (drill 1.016)
-      (layers *.Cu *.Mask F.SilkS)
+      (layers *.Cu *.Mask B.SilkS)
       (net 2 N-000001)
     )
@@
     )
     (fp_circle (center 0 0) (end 4.5 0) (layer F.SilkS) (width 0.15))
-    (pad 1 thru_hole circle (at 0 0) (size 6 6) (drill 3.2)
+    (pad "" np_thru_hole circle (at 0 0) (size 3.2 3.2) (drill 3.2)
       (layers *.Cu *.Mask F.SilkS)
     )
@@
     )
     (fp_circle (center 0 0) (end 4.5 0) (layer F.SilkS) (width 0.15))
-    (pad 1 thru_hole circle (at 0 0) (size 6 6) (drill 3.2)
+    (pad "" np_thru_hole circle (at 0 0) (size 3.2 3.2) (drill 3.2)
       (layers *.Cu *.Mask F.SilkS)
     )
@@
     (descr "DC Barrel Jack, 2.1x5.5mm")
     (tags "Power Jack")
-    (fp_text reference CON1 (at -7.62 5.461 180) (layer F.SilkS)
+    (fp_text reference CON1 (at -11.938 -3.81 180) (layer F.SilkS)
       (effects (font (size 0.762 0.762) (thickness 0.1524)))
     )
@@
       (effects (font (size 1.016 1.016) (thickness 0.2032)))
     )
-    (fp_text user 2.1x5.5mm (at -2.54 -5.715 180) (layer F.SilkS)
+    (fp_text user 2.1x5.5mm (at -2.54 -5.588 180) (layer F.SilkS)
       (effects (font (size 0.762 0.762) (thickness 0.1524)))
     )
@@
       (xy -1.21158 1.79578)) (layer F.SilkS) (width 0.00254))
   )
+  (gr_text GND (at 219.71 196.85 90) (layer B.SilkS)
+    (effects (font (size 0.762 0.762) (thickness 0.1524)) (justify left mirror))
+  )
+  (gr_text GND (at 222.25 196.85 90) (layer B.SilkS)
+    (effects (font (size 0.762 0.762) (thickness 0.1524)) (justify left mirror))
+  )
+  (gr_text "RX\n(Your TX)" (at 216.535 196.85 90) (layer B.SilkS)
+    (effects (font (size 0.762 0.762) (thickness 0.1524)) (justify left mirror))
+  )
+  (gr_text "TX\n(Your RX)" (at 224.155 196.85 90) (layer B.SilkS)
+    (effects (font (size 0.762 0.762) (thickness 0.1524)) (justify left mirror))
+  )
+  (gr_text Force- (at 223.52 162.56 90) (layer B.SilkS)
+    (effects (font (size 0.762 0.762) (thickness 0.1524)) (justify left mirror))
+  )
+  (gr_text Force+ (at 220.98 162.56 90) (layer B.SilkS)
+    (effects (font (size 0.762 0.762) (thickness 0.1524)) (justify left mirror))
+  )
+  (gr_text Sense- (at 226.06 162.56 90) (layer B.SilkS)
+    (effects (font (size 0.762 0.762) (thickness 0.1524)) (justify left mirror))
+  )
+  (gr_text Sense+ (at 218.44 162.56 90) (layer B.SilkS)
+    (effects (font (size 0.762 0.762) (thickness 0.1524)) (justify left mirror))
+  )
+  (gr_text "9V to 24V DC" (at 242.189 164.084) (layer F.SilkS)
+    (effects (font (size 0.762 0.762) (thickness 0.1524)))
+  )
   (gr_circle (center 220.98 169.545) (end 255.016 169.545) (layer Edge.Cuts) (width 0.1))
   (gr_text V- (at 197.485 170.815) (layer F.SilkS)
@@
     (effects (font (size 0.762 0.762) (thickness 0.1524)) (justify left))
   )
-  (gr_text "(v1)" (at 237.49 156.21) (layer F.SilkS)
+  (gr_text "(v2)" (at 237.49 156.21) (layer F.SilkS)
     (effects (font (size 1.016 1.016) (thickness 0.2032)) (justify left))
   )
