File: RegMouthJarPCBA/VoltagesBreakout.sch (KiCad schematic (older format))
At the start: 13 parts

Commit message: adding kelvin breakout board (v1)
Parts:
- gave numbers to parts that had none: 13
Changed lines of the file:
@@
 $EndDescr
 $Comp
-L 8P8C J?
+L 8P8C J1
 U 1 1 53B0C1AE
 P 4300 4500
-F 0 "J?" H 4350 5350 40  0000 C CNN
+F 0 "J1" H 4350 5350 40  0000 C CNN
 F 1 "8P8C" H 4950 5350 40  0000 C CNN
 F 2 "~" H 4600 4950 60  0000 C CNN
@@
 $EndComp
 $Comp
-L CONN_1 P?
+L CONN_1 P1
 U 1 1 53B0C20C
 P 5300 4600
-F 0 "P?" H 5380 4600 40  0000 L CNN
+F 0 "P1" H 5380 4600 40  0000 L CNN
 F 1 "CONN_1" H 5300 4655 30  0001 C CNN
 F 2 "" H 5300 4600 60  0000 C CNN
@@
 $EndComp
 $Comp
-L CONN_1 P?
+L CONN_1 P2
 U 1 1 53B0C21B
 P 5300 4700
-F 0 "P?" H 5380 4700 40  0000 L CNN
+F 0 "P2" H 5380 4700 40  0000 L CNN
 F 1 "CONN_1" H 5300 4755 30  0001 C CNN
 F 2 "" H 5300 4700 60  0000 C CNN
@@
 $EndComp
 $Comp
-L CONN_1 P?
+L CONN_1 P3
 U 1 1 53B0C22A
 P 5300 4800
-F 0 "P?" H 5380 4800 40  0000 L CNN
+F 0 "P3" H 5380 4800 40  0000 L CNN
 F 1 "CONN_1" H 5300 4855 30  0001 C CNN
 F 2 "" H 5300 4800 60  0000 C CNN
@@
 $EndComp
 $Comp
-L CONN_1 P?
+L CONN_1 P4
 U 1 1 53B0C239
 P 5300 4900
-F 0 "P?" H 5380 4900 40  0000 L CNN
+F 0 "P4" H 5380 4900 40  0000 L CNN
 F 1 "CONN_1" H 5300 4955 30  0001 C CNN
 F 2 "" H 5300 4900 60  0000 C CNN
@@
 $EndComp
 $Comp
-L CONN_1 P?
+L CONN_1 P5
 U 1 1 53B0C248
 P 5300 5000
-F 0 "P?" H 5380 5000 40  0000 L CNN
+F 0 "P5" H 5380 5000 40  0000 L CNN
 F 1 "CONN_1" H 5300 5055 30  0001 C CNN
 F 2 "" H 5300 5000 60  0000 C CNN
@@
 $EndComp
 $Comp
-L CONN_1 P?
+L CONN_1 P6
 U 1 1 53B0C257
 P 5300 5100
-F 0 "P?" H 5380 5100 40  0000 L CNN
+F 0 "P6" H 5380 5100 40  0000 L CNN
 F 1 "CONN_1" H 5300 5155 30  0001 C CNN
 F 2 "" H 5300 5100 60  0000 C CNN
@@
 $EndComp
 $Comp
-L CONN_1 P?
+L CONN_1 P7
 U 1 1 53B0C266
 P 5300 5200
-F 0 "P?" H 5380 5200 40  0000 L CNN
+F 0 "P7" H 5380 5200 40  0000 L CNN
 F 1 "CONN_1" H 5300 5255 30  0001 C CNN
 F 2 "" H 5300 5200 60  0000 C CNN
@@
 $EndComp
 $Comp
-L CONN_1 P?
+L CONN_1 P8
 U 1 1 53B0C275
 P 5300 5300
-F 0 "P?" H 5380 5300 40  0000 L CNN
+F 0 "P8" H 5380 5300 40  0000 L CNN
 F 1 "CONN_1" H 5300 5355 30  0001 C CNN
 F 2 "" H 5300 5300 60  0000 C CNN
@@
 	5050 5300 5150 5300
 $Comp
-L HOLE H?
+L HOLE H1
 U 1 1 53B0C2D1
 P 5750 4000
-F 0 "H?" H 5750 4055 30  0000 C CNN
+F 0 "H1" H 5750 4055 30  0000 C CNN
 F 1 "HOLE" H 5750 3940 30  0000 C CNN
 F 2 "~" H 5750 4000 60  0000 C CNN
@@
 $EndComp
 $Comp
-L HOLE H?
+L HOLE H2
 U 1 1 53B0C2E0
 P 5900 4000
-F 0 "H?" H 5900 4055 30  0000 C CNN
+F 0 "H2" H 5900 4055 30  0000 C CNN
 F 1 "HOLE" H 5900 3940 30  0000 C CNN
 F 2 "~" H 5900 4000 60  0000 C CNN
@@
 $EndComp
 $Comp
-L HOLE H?
+L HOLE H3
 U 1 1 53B0C2EF
 P 6050 4000
-F 0 "H?" H 6050 4055 30  0000 C CNN
+F 0 "H3" H 6050 4055 30  0000 C CNN
 F 1 "HOLE" H 6050 3940 30  0000 C CNN
 F 2 "~" H 6050 4000 60  0000 C CNN
@@
 $EndComp
 $Comp
-L HOLE H?
+L HOLE H4
 U 1 1 53B0C308
 P 6200 4000
-F 0 "H?" H 6200 4055 30  0000 C CNN
+F 0 "H4" H 6200 4055 30  0000 C CNN
 F 1 "HOLE" H 6200 3940 30  0000 C CNN
 F 2 "~" H 6200 4000 60  0000 C CNN
