File: RegMouthJarPCBA/LM399InterfaceBoard.sch (KiCad schematic (older format))
At the start: 15 parts

Commit message: updating LM399 interface board schematic
Parts:
- removed JP? (x2): JUMPER, ~, symbol JUMPER
- removed P?: CONN_2, ~, symbol CONN_2
- added C1, C2: 10uF, ~, symbol C_EL
- added D1, D2, D3: LED, ~, symbol LED
- added H1, H2: HOLE, ~, symbol HOLE
- added JP1, JP2, JP3, JP4: JUMPER3, ~, symbol JUMPER3
- added L1: 10uH, ~, symbol INDUCTOR_SMALL
- added P10, P11, P12, P13, P14, P15, P16, P6, P8, P9: TST, ~, symbol TST
- added R1: 10, ~, symbol R_0W25
- added R10: 47k, ~, symbol R_0W25
- added R11, R5, R8: 270, ~, symbol R_0W25
- added R2: 2.2k, ~, symbol R_0W25
- added R3, R6, R9: 10k, ~, symbol R_0W25
- added R4, R7: 100k, ~, symbol R_0W25
- added RV1: 10k, ~, symbol POT_10T
- added RV2, RV3: 100k, ~, symbol POT_10T
- added U1: 78L05, ~, symbol 78L05
- added U2: TL431LP, SOT23, symbol TL431LP
- added U3: LM339, symbol LM339
- gave numbers to parts that had none: 12
Connections:
- net labels added: 2.5V, 2.9V, 290mV, 29V, 29mV, 5V, Oven-
- wire segments 60 -> 129
- no-connect marks 0 -> 4
Other:
- note added: "1.1mA"
- note added: "Adjustment range (H+ = 40V): 37.5V to 12V"
- note added: "Adjustment range: 30V to 33V"
- note added: "Adjustment range: 8.6V to 4.3V"
- note added: "Interfaces"
- note added: "Low battery warning lamps"
- note added: "Pinout:\n1: RX (Your TX)\n2: GND\n3: GND\n4: TX (Your RX)"
- note added: "Rail limits:\n\n36V must not exceed 40 Volts (LTC2057 limit).\n\n9V must not exceed 40 Volts (LTC2057 limit).\n\nH+ must not exceed 40 Volts (LM399 limit).\n\nOven+ rail must not exceed 35 Volts (LM7805 limit)."
- note added: "Supply routing"
- note added: "Supply routing options:\n\nFor fully independent rails, use no jumpers, and supply CON1, CON2, CON3 and CON4.\n\nTo operate the 9V rail from the 36V rail, use JP1 and disconnect CON2.\n\nTo operate the 9V and H+ rails from the 36V rail, use JP1 and JP2 and disconnect CON2 and CON3.\n\nTo operate the H+ rail from the Oven+ rail, use JP3 and JP4 and disconnect CON3."
- note removed: "Pinout:\n1: My RX, Your TX\n2: GND\n3: GND\n4: My TX, Your RX"
- moved on the sheet: CON1, CON2, CON3, CON4, J1, J2, P1, P2, P3, P4, P5, P7
