File: RegMouthJarPCBA/resistor_plate.sch (KiCad schematic (older format))
At the start: 4 parts, among them P1 CONN_4

Commit message: adding kelvin breakout board (v1)
Other:
- note added: "Pinout:\n1: Sense+\n2: Force+\n3: Force-\n4: Sense-"
Changed lines of the file:
@@
 Sheet 1 1
 Title "noname.sch"
-Date "7 jun 2014"
+Date "30 jun 2014"
 Rev ""
 Comp ""
@@
 	1    0    0    -1
 $EndComp
+Text Notes 5900 2850 0    40   ~ 0
+Pinout:\n1: Sense+\n2: Force+\n3: Force-\n4: Sense-
 $EndSCHEMATC

Commit message: updating resistor board to v3.
Parts:
- removed R1: R, ~, symbol R
- added R1, R2, R3, R4: R, ~, symbol R_FOIL
Connections:
- wire segments 14 -> 15
Changed lines of the file:
@@
 Sheet 1 1
 Title "noname.sch"
-Date "30 jun 2014"
+Date "9 jul 2014"
 Rev ""
 Comp ""
@@
 Comment4 ""
 $EndDescr
-$Comp
-L R R1
-U 1 1 53929CA6
-P 5500 3650
-F 0 "R1" V 5580 3650 40  0000 C CNN
-F 1 "R" V 5507 3651 40  0000 C CNN
-F 2 "~" V 5430 3650 30  0000 C CNN
-F 3 "~" H 5500 3650 30  0000 C CNN
-	1    5500 3650
-	0    -1   -1   0
-$EndComp
 $Comp
 L CONN_4 P1
@@
 	5450 3400 5250 3400
 Wire Wire Line
-	5250 3400 5250 3750
-Wire Wire Line
 	5550 3150 5550 3400
 Wire Wire Line
 	5550 3400 5750 3400
-Wire Wire Line
-	5750 3400 5750 3750
 Wire Wire Line
 	5350 3150 5350 3300
@@
 Wire Wire Line
 	5150 3750 5250 3750
-Connection ~ 5250 3650
 Wire Wire Line
 	5650 3150 5650 3300
@@
 Wire Wire Line
 	5850 3750 5750 3750
-Connection ~ 5750 3650
 $Comp
 L HOLE H1
@@
 Text Notes 5900 2850 0    40   ~ 0
 Pinout:\n1: Sense+\n2: Force+\n3: Force-\n4: Sense-
+Wire Wire Line
+	5250 3750 5250 3400
+Wire Wire Line
+	5750 3750 5750 3400
+Connection ~ 5250 3550
+Connection ~ 5750 3550
+Wire Wire Line
+	5250 4250 5750 4250
+$Comp
+L R_FOIL R3
+U 1 1 53BCC05E
+P 5500 3750
+F 0 "R3" V 5580 3750 40  0000 C CNN
+F 1 "R" V 5507 3751 40  0000 C CNN
+F 2 "~" V 5430 3750 30  0000 C CNN
+F 3 "~" H 5500 3750 30  0000 C CNN
+	1    5500 3750
+	0    -1   -1   0
+$EndComp
+$Comp
+L R_FOIL R2
+U 1 1 53BCC0CB
+P 5500 3550
+F 0 "R2" V 5580 3550 40  0000 C CNN
+F 1 "R" V 5507 3551 40  0000 C CNN
+F 2 "~" V 5430 3550 30  0000 C CNN
+F 3 "~" H 5500 3550 30  0000 C CNN
+	1    5500 3550
+	0    -1   -1   0
+$EndComp
+$Comp
+L R_FOIL R1
+U 1 1 53BCC0D1
+P 5250 4000
+F 0 "R1" V 5330 4000 40  0000 C CNN
+F 1 "R" V 5257 4001 40  0000 C CNN
+F 2 "~" V 5180 4000 30  0000 C CNN
+F 3 "~" H 5250 4000 30  0000 C CNN
+	1    5250 4000
+	-1   0    0    1
+$EndComp
+$Comp
+L R_FOIL R4
+U 1 1 53BCC0D7
+P 5750 4000
+F 0 "R4" V 5830 4000 40  0000 C CNN
+F 1 "R" V 5757 4001 40  0000 C CNN
+F 2 "~" V 5680 4000 30  0000 C CNN
+F 3 "~" H 5750 4000 30  0000 C CNN
+	1    5750 4000
+	-1   0    0    1
+$EndComp
 $EndSCHEMATC
